File: PCB/PowerBank_PCB.kicad_pcb (KiCad board)
At the start: 2 copper layers, 261 x 92 mm, 38 parts, among them J1 USB_C_Receptacle_PowerOnly_6P, J10 SSD1306, J2 Conn_01x02, J3 Conn_01x02, J4 Conn_01x02, J5 Conn_01x02, J6 Conn_01x02, J7 Conn_01x02, J8 Conn_01x02, J9 Conn_01x02

Commit message: Added Correct Footprints
The Schematic is now completed with the correct Foot Prints
Parts:
- removed REF** (x4): MountingHole_3.2mm_M3, MountingHole:MountingHole_3.2mm_M3
- removed REF**: SW_TL6340AF160Q, Library:SW_TL6340AF160Q
- added C10: 1u, Capacitor_SMD:C_1206_3216Metric_Pad1.33x1.80mm_HandSolder, F.Cu at (160.2, 27.9)
- added C7: 1n, Capacitor_SMD:C_1206_3216Metric_Pad1.33x1.80mm_HandSolder, F.Cu at (150.2, 27.9)
- added C8: 10u, Capacitor_SMD:C_1206_3216Metric_Pad1.33x1.80mm_HandSolder, F.Cu at (153.6, 27.9)
- added C9: 10u, Capacitor_SMD:C_1206_3216Metric_Pad1.33x1.80mm_HandSolder, F.Cu at (156.9, 27.9)
- added Q2: Q_PMOS_GSD, Package_TO_SOT_SMD:SOT-23_Handsoldering, F.Cu at (200.4, 35.0)
- added Q3: MMBT3906, Package_TO_SOT_SMD:SOT-23_Handsoldering, F.Cu at (205.2, 35.0)
- added Q4: Q_PMOS_GSD, Package_TO_SOT_SMD:SOT-23_Handsoldering, F.Cu at (209.9, 35.0)
- added R10: 10k, Resistor_SMD:R_1206_3216Metric_Pad1.30x1.75mm_HandSolder, F.Cu at (179.6, 29.3)
- added R3: 1k, Resistor_SMD:R_1206_3216Metric_Pad1.30x1.75mm_HandSolder, F.Cu at (176.3, 35.3)
- added R6: 10k, Resistor_SMD:R_1206_3216Metric_Pad1.30x1.75mm_HandSolder, F.Cu at (186.2, 35.3)
- added R7: 100k, Resistor_SMD:R_1206_3216Metric_Pad1.30x1.75mm_HandSolder, F.Cu at (169.7, 29.3)
- added R8: 10k, Resistor_SMD:R_1206_3216Metric_Pad1.30x1.75mm_HandSolder, F.Cu at (173.0, 29.3)
- added R9: 2, Resistor_SMD:R_1206_3216Metric_Pad1.30x1.75mm_HandSolder, F.Cu at (176.3, 29.3)
- added S1: TL6340AF160Q, Custom_FootPrints:SW_TL6340AF160Q, F.Cu at (47.6, 44.1)
- J1: footprint Connector_USB:USB_C_Receptacle_GCT_USB4110 -> Connector_USB:USB_C_Receptacle_GCT_USB4125-xx-x_6P_TopMnt_Horizontal
- U1: value ~ -> IP5310
- moved D1 265.6 mm to (214.5, 33.2), turned to 90 degrees
- moved J1 242.6 mm to (193.2, 31.0)
- moved J10 239.7 mm to (200.2, 29.5), turned to 90 degrees
- moved J5 226.5 mm to (126.3, 108.5), turned to 90 degrees
- moved J6 213.7 mm to (149.0, 108.5), turned to 90 degrees
- moved J4 198.2 mm to (103.6, 108.5), turned to 90 degrees
- moved J7 189.7 mm to (171.7, 108.5), turned to 90 degrees
- moved U1 178.2 mm to (228.2, 34.2), turned to 90 degrees
- moved J3 171.0 mm to (80.9, 108.5), turned to 90 degrees
- moved L1 170.7 mm to (220.7, 34.0), turned to 90 degrees
- moved J8 168.2 mm to (194.4, 108.5), turned to 90 degrees
- moved R4 151.6 mm to (179.6, 35.3)
- moved J9 150.3 mm to (217.1, 108.5), turned to 90 degrees
- moved R5 150.1 mm to (182.9, 35.3), turned to 90 degrees
- moved F4 147.0 mm to (145.8, 34.6), turned to 90 degrees
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Connections:
- A1 pad 13: GND -> Net-(J10-GND)
- A1 pad 18: GND -> Net-(J10-GND)
- A1 pad 23: GND -> Net-(J10-GND)
- A1 pad 28: GND -> Net-(J10-GND)
- A1 pad 3: GND -> Net-(J10-GND)
- A1 pad 38: GND -> Net-(J10-GND)
- A1 pad 8: GND -> Net-(J10-GND)
- A1 pad D2: GND -> Net-(J10-GND)
- J1 pad A9: Net-(D1-K) -> Net-(Q2-D)
- J1 pad B9: Net-(D1-K) -> Net-(Q2-D)
- J10 pad 4: GND -> Net-(J10-GND)
- R2 pad 2: GND -> Net-(J10-GND)
- U1 pad 10: Net-(D1-K) -> Net-(Q4-S)
- U1 pad 11: unconnected-(U1-VBUSG-Pad11) -> Net-(U1-VBUSG)
- U1 pad 23: Net-(D1-K) -> Net-(Q2-D)
- U1 pad 24: Net-(D1-K) -> Net-(Q2-D)
- U1 pad 4: (no net) -> unconnected-(U1-VTHS-Pad4)
Routing:
- net GND: track 620.1 -> 0.00 mm, vias 4 -> 0
- net /BAT+: track 197.9 -> 0.00 mm
- net /SDA: track 187.5 -> 0.00 mm, vias 2 -> 0
- net Net-(D1-K): track 177.8 -> 0.00 mm, vias 6 -> 0
- net /SCL: track 171.5 -> 0.00 mm, vias 2 -> 0
- net Net-(J1-CC1): track 159.5 -> 0.00 mm, vias 2 -> 0
- net Net-(J1-CC2): track 159.5 -> 0.00 mm, vias 2 -> 0
- net Net-(U1-KEY): track 150.3 -> 0.00 mm, vias 2 -> 0
- net /VCC: track 145.8 -> 0.00 mm
- net /ADC: track 45.2 -> 0.00 mm, vias 2 -> 0
- net Net-(U1-NTC): track 14.0 -> 0.00 mm
- net Net-(C4-Pad1): track 9.07 -> 0.00 mm
- net Net-(C3-Pad1): track 7.38 -> 0.00 mm
- net Net-(L1-Pad1): track 6.85 -> 0.00 mm
- net Net-(J2-Pin_1): track 5.83 -> 0.00 mm
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- added copper zone on F.Cu, net (none)
- removed copper zone on B.Cu, net (none)
Other:
- board size 261 x 92 mm -> 183.5 x 96.2 mm
- copper layers 2 -> 4
- board text added: "Power Bank PCB Design"
- board text added: "V1.0"
