File: PCB/PowerBank_PCB.kicad_sch (KiCad schematic)
At the start: 34 parts, among them J1 USB_C_Receptacle_PowerOnly_6P, J10 SSD1306, J2 Conn_01x02, J3 Conn_01x02, J4 Conn_01x02, J5 Conn_01x02, J6 Conn_01x02, J7 Conn_01x02, J8 Conn_01x02, J9 Conn_01x02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

Commit message: Implemented proper Circuit for USB-C Input/Output
Implemented PMOS transistors to provide USB-C Input/Output functionalities
Parts:
- added C10: 1u, symbol Device:C
- added C7: 1n, symbol Device:C
- added C8, C9: 10u, symbol Device:C
- added Q1: PNP, symbol Simulation_SPICE:PNP
- added Q2, Q4: Q_PMOS_GSD, symbol Transistor_FET:Q_PMOS_GSD
- added R10, R6, R8: 10k, symbol Device:R_Small_US
- added R3: 1k, symbol Device:R_Small_US
- added R7: 100k, symbol Device:R_Small_US
- added R9: 2, symbol Device:R_Small_US
Connections:
- net GND: now also C8.2, C9.2, R8.2
- net at J1.A9 (VBUS), J1.B9 (VBUS), U1.23 (VIN)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: now also Q2.3 (D), Q4.3 (D); no longer D1.1 (K), U1.10 (VBUS)
- net at U1.11 (VBUSG): now also C10.2, R10.2
- new net: C9.1, Q2.2 (S), R9.1
- new net: C8.1, R9.2
- new net: C7.2, Q1.1 (C), R7.2, R8.1
- new net: Q1.2 (B), R6.2
- new net: C7.1, Q1.3 (E), Q2.1 (G), R3.1, R7.1
- new net: C10.1, Q4.1 (G), R10.1
- new net: Q4.2 (S), U1.10 (VBUS)
- new net: D1.1 (K), R3.2, R6.1
Other:
- moved on the sheet: A1, C1, C2, C3, C4, C5, C6, D1, F1, F2, F3, F4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

Commit message: Added Correct Footprints
The Schematic is now completed with the correct Foot Prints
Parts:
- removed Q1: PNP, symbol Simulation_SPICE:PNP
- added Q3: MMBT3906, Package_TO_SOT_SMD:SOT-23_Handsoldering, symbol Transistor_BJT:MMBT3906
- C10, C7, C8, C9: footprint (none) -> Capacitor_SMD:C_1206_3216Metric_Pad1.33x1.80mm_HandSolder
- J1: footprint Connector_USB:USB_C_Receptacle_GCT_USB4110 -> Connector_USB:USB_C_Receptacle_GCT_USB4125-xx-x_6P_TopMnt_Horizontal
- Q2, Q4: footprint (none) -> Package_TO_SOT_SMD:SOT-23_Handsoldering
- R10, R3, R6, R7, R8, R9: footprint (none) -> Resistor_SMD:R_1206_3216Metric_Pad1.30x1.75mm_HandSolder
- S1: footprint TL6340AF160Q:SW_TL6340AF160Q -> Custom_FootPrints:SW_TL6340AF160Q
Connections:
- net GND: now also J1.SH (SHIELD); no longer J1.S1 (SHIELD)
- net at C7.2, R7.2, R8.1: now also Q3.3 (C)
- net at R6.2: now also Q3.1 (B)
- net at C7.1, Q2.1 (G), R3.1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: now also Q3.2 (E)
Other:
- note added: "6/16/2026"
- note added: "Power Bank Schematic"
- note added: "V1.0"
